File: ap63300.kicad_sch (KiCad schematic)
At the start: 8 parts

Commit message: Annotate
Parts:
- gave numbers to parts that had none: 1
Changed lines of the file:
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@@
   (symbol (lib_id "AP63300WU-7:AP63300WU-7") (at 67.31 43.18 0) (unit 1)
     (in_bom yes) (on_board yes) (fields_autoplaced)
-    (property "Reference" "U?" (id 0) (at 67.31 29.3202 0))
+    (property "Reference" "U1" (id 0) (at 67.31 29.3202 0))
     (property "Value" "AP63300WU-7" (id 1) (at 67.31 31.8571 0))
     (property "Footprint" "AP63300WU-7:SOT95P280X100-6N" (id 2) (at 72.39 20.32 0)
