File: pink_panda.kicad_sch (KiCad schematic)
At the start: 2 parts

Commit message: Annotate
Parts:
- gave numbers to parts that had none: 2
Changed lines of the file:
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@@
   (symbol (lib_id "Connector:Conn_01x12_Female") (at 38.1 35.56 0) (unit 1)
     (in_bom yes) (on_board yes)
-    (property "Reference" "J?" (id 0) (at 38.8112 35.9953 0)
+    (property "Reference" "J3" (id 0) (at 38.8112 35.9953 0)
       (effects (font (size 1.27 1.27)) (justify left))
     )
@@
   (symbol (lib_id "Connector:Conn_01x12_Female") (at 68.58 38.1 0) (unit 1)
     (in_bom yes) (on_board yes) (fields_autoplaced)
-    (property "Reference" "J?" (id 0) (at 69.2912 38.5353 0)
+    (property "Reference" "J4" (id 0) (at 69.2912 38.5353 0)
       (effects (font (size 1.27 1.27)) (justify left))
     )

Commit message: Import parts to pcb
Parts:
- J3: value Conn_01x12_Female -> Left
- J4: value Conn_01x12_Female -> Right
Changed lines of the file:
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@@
       (effects (font (size 1.27 1.27)) (justify left))
     )
-    (property "Value" "Conn_01x12_Female" (id 1) (at 38.8112 38.5322 0)
+    (property "Value" "Left" (id 1) (at 38.8112 38.5322 0)
       (effects (font (size 1.27 1.27)) (justify left) hide)
     )
@@
       (effects (font (size 1.27 1.27)) (justify left))
     )
-    (property "Value" "Conn_01x12_Female" (id 1) (at 69.2912 41.0722 0)
+    (property "Value" "Right" (id 1) (at 69.2912 41.0722 0)
       (effects (font (size 1.27 1.27)) (justify left) hide)
     )
